Commit message: Update Horst900_urdf.urdf
new urdf created with correct origin

File: Horst900_urdf.urdf (robot description, URDF)
Before this commit: robot Horst900_urdf, 7 links, 6 joints
Links:
- link Link1: mass 0.06735 -> 0.0673503751305048
- link Link2: mass 0.22367 -> 0.223671456970964
- link Link3: mass 0.25309 -> 0.253092969796525
- link Link4: mass 0.038503 -> 0.0385025243577973
- link Link5: mass 0.025507 -> 0.0255070628905158
- link Link6: mass 1.8181 -> 1.81808855431787
- link base_link: mass 1.21 -> 1.20995872182931
Joints:
- joint Joint1: axis 0 1 0 -> 0 0 1; origin xyz=0.02505 -0.3825 2.8818E-05 rpy=1.57079632679 0 0 -> xyz=0.02505 2.8818E-05 0.3825 rpy=1.5708 0 0
- joint Joint2: axis 0 0 -1 -> 0 0 1
- joint Joint3: axis 1 0 0 -> 0 0 1
- joint Joint5: axis 0 0 -1 -> 0 0 1
- joint Joint6: axis 0 0 -1 -> 0 0 1
