Commit message: Right urdf File
URDF File changed and CAD model

File: Horst900_Attemp2.urdf (robot description, URDF)
Before this commit: robot Horst900_urdf, 7 links, 6 joints
Links:
- removed link Link1
- removed link Link2
- removed link Link3
- removed link Link4
- removed link Link5
- removed link Link6
- added link link1, mass 0.06735; collision mesh filename=package://Horst900_Attemp2/meshes/link1.STL; visual mesh filename=package://Horst900_Attemp2/meshes/link1.STL
- added link link2, mass 0.22367; collision mesh filename=package://Horst900_Attemp2/meshes/link2.STL; visual mesh filename=package://Horst900_Attemp2/meshes/link2.STL
- added link link3, mass 0.25309; collision mesh filename=package://Horst900_Attemp2/meshes/link3.STL; visual mesh filename=package://Horst900_Attemp2/meshes/link3.STL
- added link link4, mass 0.038503; collision mesh filename=package://Horst900_Attemp2/meshes/link4.STL; visual mesh filename=package://Horst900_Attemp2/meshes/link4.STL
- added link link5, mass 0.025507; collision mesh filename=package://Horst900_Attemp2/meshes/link5.STL; visual mesh filename=package://Horst900_Attemp2/meshes/link5.STL
- added link link6, mass 1.8181; collision mesh filename=package://Horst900_Attemp2/meshes/link6.STL; visual mesh filename=package://Horst900_Attemp2/meshes/link6.STL
- link base_link: mass 1.20995872182931 -> 1.21; geometry collision mesh filename=package://Horst900_Attemp2/meshes/base_link.STL; visual mesh filename=package://Horst900_Attemp2/meshes/base_link.STL
Joints:
- removed joint Joint1
- removed joint Joint2
- removed joint Joint3
- removed joint Joint4
- removed joint Joint5
- removed joint Joint6
- added joint joint1: type revolute, parent base_link, child link1, origin xyz=0 0 0.0565 rpy=1.5708 0 0, axis 0 -1 0, limit lower=0 upper=0 effort=0 velocity=0
- added joint joint2: type revolute, parent link1, child link2, origin xyz=0.05675 0.28257 0 rpy=0 0 0, axis 0 0 1, limit lower=0 upper=0 effort=0 velocity=0
- added joint joint3: type revolute, parent link2, child link3, origin xyz=6.7742E-05 0.407 0 rpy=0 1.5708 0, axis 1 0 0, limit lower=0 upper=0 effort=0 velocity=0
- added joint joint4: type revolute, parent link3, child link4, origin xyz=-2.4956E-05 0.03648 0.12703 rpy=0 1.5708 0, axis 1 0 0, limit lower=0 upper=0 effort=0 velocity=0
- added joint joint5: type revolute, parent link4, child link5, origin xyz=-0.308 0 0 rpy=-1.5708 0 3.1416, axis 0 1 0, limit lower=0 upper=0 effort=0 velocity=0
- added joint joint6: type revolute, parent link5, child link6, origin xyz=0.0001 -0.0002 0 rpy=0 0 3.1416, axis 0 0 -1, limit lower=0 upper=0 effort=0 velocity=0

File: Horst900_Attemp2/urdf/Horst900_Attemp2.urdf (robot description, URDF)
Before this commit: robot Horst900_urdf, 7 links, 6 joints
Links:
- removed link Link1
- removed link Link2
- removed link Link3
- removed link Link4
- removed link Link5
- removed link Link6
- added link link1, mass 0.06735; collision mesh filename=package://Horst900_Attemp2/meshes/link1.STL; visual mesh filename=package://Horst900_Attemp2/meshes/link1.STL
- added link link2, mass 0.22367; collision mesh filename=package://Horst900_Attemp2/meshes/link2.STL; visual mesh filename=package://Horst900_Attemp2/meshes/link2.STL
- added link link3, mass 0.25309; collision mesh filename=package://Horst900_Attemp2/meshes/link3.STL; visual mesh filename=package://Horst900_Attemp2/meshes/link3.STL
- added link link4, mass 0.038503; collision mesh filename=package://Horst900_Attemp2/meshes/link4.STL; visual mesh filename=package://Horst900_Attemp2/meshes/link4.STL
- added link link5, mass 0.025507; collision mesh filename=package://Horst900_Attemp2/meshes/link5.STL; visual mesh filename=package://Horst900_Attemp2/meshes/link5.STL
- added link link6, mass 1.8181; collision mesh filename=package://Horst900_Attemp2/meshes/link6.STL; visual mesh filename=package://Horst900_Attemp2/meshes/link6.STL
- link base_link: geometry collision mesh filename=package://Horst900_Attemp2/meshes/base_link.STL; visual mesh filename=package://Horst900_Attemp2/meshes/base_link.STL
Joints:
- removed joint Joint1
- removed joint Joint2
- removed joint Joint3
- removed joint Joint4
- removed joint Joint5
- removed joint Joint6
- added joint joint1: type revolute, parent base_link, child link1, origin xyz=0 0 0.0565 rpy=1.5708 0 0, axis 0 -1 0, limit lower=0 upper=0 effort=0 velocity=0
- added joint joint2: type revolute, parent link1, child link2, origin xyz=0.05675 0.28257 0 rpy=0 0 0, axis 0 0 1, limit lower=0 upper=0 effort=0 velocity=0
- added joint joint3: type revolute, parent link2, child link3, origin xyz=6.7742E-05 0.407 0 rpy=0 1.5708 0, axis 1 0 0, limit lower=0 upper=0 effort=0 velocity=0
- added joint joint4: type revolute, parent link3, child link4, origin xyz=-2.4956E-05 0.03648 0.12703 rpy=0 1.5708 0, axis 1 0 0, limit lower=0 upper=0 effort=0 velocity=0
- added joint joint5: type revolute, parent link4, child link5, origin xyz=-0.308 0 0 rpy=-1.5708 0 3.1416, axis 0 1 0, limit lower=0 upper=0 effort=0 velocity=0
- added joint joint6: type revolute, parent link5, child link6, origin xyz=0.0001 -0.0002 0 rpy=0 0 3.1416, axis 0 0 -1, limit lower=0 upper=0 effort=0 velocity=0
